File: class02/simpleCH552_finished.brd (EAGLE design)
At the start: 40.6 x 12 mm, 15 parts, among them U2 CH552G, X1 USBPCB

Commit message: update part number
Parts:
- F1: value (none) -> DNP
- renumbered U2 to U1
Changed lines of the file:
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@@
 <attribute name="VALUE" x="16.621" y="7.7674" size="0.6096" layer="27" rot="R180"/>
 </element>
-<element name="F1" library="adafruit" library_urn="urn:adsk.eagle:library:420" package="R1206" value="" x="15.367" y="3.429" smashed="yes">
+<element name="F1" library="adafruit" library_urn="urn:adsk.eagle:library:420" package="R1206" value="DNP" x="15.367" y="3.429" smashed="yes">
 <attribute name="LCSC" value="C151162" x="48.387" y="-41.021" size="1.778" layer="27" display="off"/>
 <attribute name="VALUE" x="13.97" y="1.016" size="1.27" layer="27"/>
 </element>
 <element name="R1" library="rcl" library_urn="urn:adsk.eagle:library:334" package="R0805" package3d_urn="urn:adsk.eagle:package:23553/2" value="20K" x="31.75" y="5.9944" smashed="yes">
+<attribute name="LCSC" value="C702832" x="31.75" y="5.9944" size="1.778" layer="27" display="off"/>
 <attribute name="POPULARITY" value="85" x="48.26" y="-7.9756" size="1.778" layer="27" display="off"/>
 <attribute name="SPICEPREFIX" value="R" x="48.26" y="-7.9756" size="1.778" layer="27" display="off"/>
 </element>
 <element name="R2" library="rcl" library_urn="urn:adsk.eagle:library:334" package="R0805" package3d_urn="urn:adsk.eagle:package:23553/2" value="20K" x="31.75" y="10.5664" smashed="yes" rot="R180">
+<attribute name="LCSC" value="C702832" x="31.75" y="10.5664" size="1.778" layer="27" rot="R180" display="off"/>
 <attribute name="POPULARITY" value="85" x="-5.08" y="24.5364" size="1.778" layer="27" rot="R180" display="off"/>
 <attribute name="SPICEPREFIX" value="R" x="-5.08" y="24.5364" size="1.778" layer="27" rot="R180" display="off"/>
 </element>
-<element name="U2" library="myOwnLib" package="MY_IC_SO16" value="CH552G" x="22.86" y="5.9944" smashed="yes">
+<element name="U1" library="myOwnLib" package="MY_IC_SO16" value="CH552G" x="22.86" y="5.9944" smashed="yes">
 <attribute name="LCSC" value="C111292" x="50.8" y="2.1844" size="1.778" layer="27" display="off"/>
 <attribute name="VALUE" x="18.796" y="5.3594" size="1.27" layer="27" ratio="10"/>
 </element>
-<element name="LED1" library="BeagleBone_Black_Wireless" library_urn="urn:adsk.eagle:library:6644236" package="GHI-BASICCOMPONENTS_0805-LED" package3d_urn="urn:adsk.eagle:package:6644356/2" value="PWR" x="31.75" y="8.2804" smashed="yes" rot="R90"/>
+<element name="LED1" library="BeagleBone_Black_Wireless" library_urn="urn:adsk.eagle:library:6644236" package="GHI-BASICCOMPONENTS_0805-LED" package3d_urn="urn:adsk.eagle:package:6644356/2" value="PWR" x="31.75" y="8.2804" smashed="yes" rot="R90">
+<attribute name="LCSC" value="C389523" x="31.75" y="8.2804" size="1.778" layer="27" rot="R90" display="off"/>
+</element>
 <element name="X1" library="SparkFun" package="USB-A-PCB" value="USBPCB" x="5.207" y="5.9944" smashed="yes"/>
 <element name="J1" library="SparkFun-Connectors" library_urn="urn:adsk.eagle:library:513" package="1X07_NO_SILK" package3d_urn="urn:adsk.eagle:package:38136/1" value="" x="13.081" y="0.9144" smashed="yes">
@@
 <element name="TP2" library="SparkFun-Connectors" library_urn="urn:adsk.eagle:library:513" package="PAD.03X.04" package3d_urn="urn:adsk.eagle:package:38287/1" value="TEST-POINT3X4" x="11.938" y="7.0104" smashed="yes"/>
 <element name="S1" library="SparkFun-Switches" library_urn="urn:adsk.eagle:library:535" package="TACTILE_SWITCH_SMD_6.2MM_TALL" package3d_urn="urn:adsk.eagle:package:40172/1" value="MOMENTARY-SWITCH-SPST-SMD-6.2MM-TALL" x="37.211" y="5.9944" smashed="yes" rot="R270">
+<attribute name="LCSC" value="C557616" x="37.211" y="5.9944" size="1.778" layer="27" rot="R270" display="off"/>
 <attribute name="PROD_ID" value="SWCH-11966" x="37.211" y="5.9944" size="1.778" layer="27" rot="R270" display="off"/>
 <attribute name="SF_SKU" value="COM-12992" x="37.211" y="5.9944" size="1.778" layer="27" rot="R270" display="off"/>
 </element>
 <element name="R3" library="rcl" library_urn="urn:adsk.eagle:library:334" package="R0805" package3d_urn="urn:adsk.eagle:package:23553/2" value="20K" x="31.75" y="1.4224" smashed="yes" rot="R180">
+<attribute name="LCSC" value="C702832" x="31.75" y="1.4224" size="1.778" layer="27" rot="R180" display="off"/>
 <attribute name="POPULARITY" value="85" x="31.75" y="1.4224" size="1.778" layer="27" rot="R180" display="off"/>
 <attribute name="SPICEPREFIX" value="R" x="31.75" y="1.4224" size="1.778" layer="27" rot="R180" display="off"/>
 </element>
-<element name="LED2" library="BeagleBone_Black_Wireless" library_urn="urn:adsk.eagle:library:6644236" package="GHI-BASICCOMPONENTS_0805-LED" package3d_urn="urn:adsk.eagle:package:6644356/2" value="P3.3" x="31.75" y="3.7084" smashed="yes" rot="R90"/>
+<element name="LED2" library="BeagleBone_Black_Wireless" library_urn="urn:adsk.eagle:library:6644236" package="GHI-BASICCOMPONENTS_0805-LED" package3d_urn="urn:adsk.eagle:package:6644356/2" value="P3.3" x="31.75" y="3.7084" smashed="yes" rot="R90">
+<attribute name="LCSC" value="C389524" x="31.75" y="3.7084" size="1.778" layer="27" rot="R90" display="off"/>
+</element>
 </elements>
 <signals>
@@
 <contactref element="C1" pad="2"/>
 <contactref element="C2" pad="2"/>
-<contactref element="U2" pad="14"/>
+<contactref element="U1" pad="14"/>
 <contactref element="X1" pad="GND"/>
 <contactref element="J1" pad="1"/>
@@
 <signal name="3.3V">
 <contactref element="C2" pad="1"/>
-<contactref element="U2" pad="16"/>
+<contactref element="U1" pad="16"/>
 <wire x1="18.415" y1="8.8138" x2="16.6464" y2="8.8138" width="0.254" layer="1"/>
 <wire x1="16.6464" y1="8.8138" x2="16.621" y2="8.7884" width="0.254" layer="1"/>
 </signal>
 <signal name="USB_D-">
-<contactref element="U2" pad="13"/>
+<contactref element="U1" pad="13"/>
 <contactref element="X1" pad="USB_M"/>
 <wire x1="5.507" y1="4.9944" x2="12.2588" y2="4.9944" width="0.254" layer="1"/>
@@
 </signal>
 <signal name="USB_D+">
-<contactref element="U2" pad="12"/>
+<contactref element="U1" pad="12"/>
 <contactref element="R1" pad="1"/>
 <contactref element="X1" pad="USB_P"/>
@@
 </signal>
 <signal name="P1.1">
-<contactref element="U2" pad="9"/>
+<contactref element="U1" pad="9"/>
 <contactref element="J1" pad="2"/>
 <wire x1="15.621" y1="0.9144" x2="18.669" y2="3.9624" width="0.2032" layer="16"/>
@@
 <contactref element="F1" pad="2"/>
 <contactref element="C1" pad="1"/>
-<contactref element="U2" pad="15"/>
+<contactref element="U1" pad="15"/>
 <contactref element="R2" pad="1"/>
 <contactref element="F1" pad="1"/>
@@
 </signal>
 <signal name="P1.4">
-<contactref element="U2" pad="2"/>
+<contactref element="U1" pad="2"/>
 <contactref element="J1" pad="3"/>
 <wire x1="19.685" y1="3.175" x2="19.685" y2="2.4384" width="0.2032" layer="1"/>
@@
 </signal>
 <signal name="P1.5">
-<contactref element="U2" pad="3"/>
+<contactref element="U1" pad="3"/>
 <contactref element="J1" pad="4"/>
 <wire x1="20.955" y1="3.175" x2="20.955" y2="1.1684" width="0.2032" layer="1"/>
@@
 </signal>
 <signal name="P1.6">
-<contactref element="U2" pad="4"/>
+<contactref element="U1" pad="4"/>
 <contactref element="J1" pad="5"/>
 <wire x1="22.225" y1="3.175" x2="22.225" y2="1.9304" width="0.2032" layer="1"/>
@@
 </signal>
 <signal name="P1.7">
-<contactref element="U2" pad="5"/>
+<contactref element="U1" pad="5"/>
 <contactref element="J1" pad="6"/>
 <wire x1="23.495" y1="3.175" x2="23.495" y2="2.54" width="0.2032" layer="1"/>
@@
 </signal>
 <signal name="P3.4">
-<contactref element="U2" pad="11"/>
+<contactref element="U1" pad="11"/>
 <contactref element="J2" pad="7"/>
 <wire x1="24.765" y1="8.8138" x2="24.765" y2="8.1026" width="0.2032" layer="1"/>
@@
 </signal>
 <signal name="P3.3">
-<contactref element="U2" pad="10"/>
+<contactref element="U1" pad="10"/>
 <contactref element="J2" pad="6"/>
 <wire x1="26.035" y1="8.8138" x2="26.035" y2="10.8204" width="0.2032" layer="1"/>
@@
 </signal>
 <signal name="P3.2">
-<contactref element="U2" pad="1"/>
+<contactref element="U1" pad="1"/>
 <contactref element="J2" pad="5"/>
 <wire x1="18.415" y1="3.175" x2="18.415" y2="3.937" width="0.2032" layer="1"/>
@@
 </signal>
 <signal name="P3.1">
-<contactref element="U2" pad="7"/>
+<contactref element="U1" pad="7"/>
 <contactref element="J2" pad="4"/>
 <via x="21.59" y="7.239" extent="1-16" drill="0.35"/>
@@
 </signal>
 <signal name="P3.0">
-<contactref element="U2" pad="8"/>
+<contactref element="U1" pad="8"/>
 <contactref element="J2" pad="3"/>
 <wire x1="18.161" y1="11.0744" x2="18.161" y2="8.89" width="0.2032" layer="16"/>
@@
 </signal>
 <signal name="RST">
-<contactref element="U2" pad="6"/>
+<contactref element="U1" pad="6"/>
 <contactref element="J1" pad="7"/>
 <wire x1="24.765" y1="3.175" x2="24.765" y2="3.8862" width="0.2032" layer="1"/>
