File: class02/simpleCH552_finished.sch (EAGLE design)
At the start: 15 parts, among them U2 CH552G, X1 USBPCB

Commit message: update part number
Parts:
- F1: value (none) -> DNP
- LED1: LCSC (none) -> C389523
- LED2: LCSC (none) -> C389524
- R1, R2, R3: LCSC (none) -> C702832
- S1: LCSC (none) -> C557616
- renumbered U2 to U1
