File: class07/atmega328_dip_board/atmega328_dip_board.sch (EAGLE design)
At the start: 9 parts, among them U1 328P

Commit message: update board
Connections:
- removed net N$21: J4.7
- removed net N$22: J4.8
- removed net N$23: J4.9
- removed net N$24: J4.10
- removed net N$25: J4.11
- removed net N$26: J4.12
- removed net N$27: J4.13
- removed net N$28: J4.14
- new net N$2: D1.A, R1.2
- net 5V: now also C1.+, J4.12, J4.8
- net A4: now also J4.13
- net A5: now also J4.14
- net AREF: now also J4.10
- net D13: now also R1.1
- net GND: now also C1.-, D1.C, J4.11, J4.7, Y1.2
- net RESET: now also J4.9
- net XTAL1: now also Y1.1
- net XTAL2: now also Y1.3
Other:
- moved on the sheet: C1, D1, R1
Changed lines of the file:
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@@
 <part name="J1" library="SparkFun-Connectors" library_urn="urn:adsk.eagle:library:513" deviceset="CONN_07" device="NO_SILK" package3d_urn="urn:adsk.eagle:package:38136/2"/>
 <part name="J2" library="SparkFun-Connectors" library_urn="urn:adsk.eagle:library:513" deviceset="CONN_07" device="NO_SILK" package3d_urn="urn:adsk.eagle:package:38136/2"/>
+<part name="SUPPLY1" library="supply2" library_urn="urn:adsk.eagle:library:372" deviceset="GND" device=""/>
+<part name="SUPPLY2" library="supply2" library_urn="urn:adsk.eagle:library:372" deviceset="GND" device=""/>
+<part name="SUPPLY3" library="supply2" library_urn="urn:adsk.eagle:library:372" deviceset="GND" device=""/>
 </parts>
 <sheets>
@@
 <attribute name="VALUE" x="17.78" y="60.452" size="1.778" layer="96" font="vector" align="bottom-center"/>
 </instance>
-<instance part="D1" gate="D1" x="5.08" y="15.24" smashed="yes">
-<attribute name="NAME" x="1.651" y="10.668" size="1.778" layer="95" font="vector" rot="R90"/>
-<attribute name="VALUE" x="6.985" y="10.668" size="1.778" layer="96" font="vector" rot="R90" align="top-left"/>
-</instance>
-<instance part="R1" gate="G$1" x="7.62" y="25.4" smashed="yes">
-<attribute name="NAME" x="7.62" y="26.924" size="1.778" layer="95" font="vector" align="bottom-center"/>
-<attribute name="VALUE" x="7.62" y="23.876" size="1.778" layer="96" font="vector" align="top-center"/>
-</instance>
-<instance part="C1" gate="G$1" x="-20.32" y="33.02" smashed="yes">
-<attribute name="NAME" x="-19.304" y="33.655" size="1.778" layer="95" font="vector"/>
-<attribute name="VALUE" x="-19.304" y="28.829" size="1.778" layer="96" font="vector"/>
+<instance part="D1" gate="D1" x="101.6" y="27.94" smashed="yes">
+<attribute name="NAME" x="98.171" y="23.368" size="1.778" layer="95" font="vector" rot="R90"/>
+<attribute name="VALUE" x="103.505" y="23.368" size="1.778" layer="96" font="vector" rot="R90" align="top-left"/>
+</instance>
+<instance part="R1" gate="G$1" x="91.44" y="30.48" smashed="yes">
+<attribute name="NAME" x="91.44" y="32.004" size="1.778" layer="95" font="vector" align="bottom-center"/>
+<attribute name="VALUE" x="91.44" y="28.956" size="1.778" layer="96" font="vector" align="top-center"/>
+</instance>
+<instance part="C1" gate="G$1" x="12.7" y="81.28" smashed="yes">
+<attribute name="NAME" x="13.716" y="81.915" size="1.778" layer="95" font="vector"/>
+<attribute name="VALUE" x="13.716" y="77.089" size="1.778" layer="96" font="vector"/>
 </instance>
 <instance part="J1" gate="J1" x="127" y="40.64" smashed="yes" rot="R180">
@@
 <attribute name="VALUE" x="154.94" y="50.546" size="1.778" layer="96" font="vector" rot="R180"/>
 <attribute name="NAME" x="154.94" y="27.432" size="1.778" layer="95" font="vector" rot="R180"/>
+</instance>
+<instance part="SUPPLY1" gate="GND" x="17.78" y="48.26" smashed="yes">
+<attribute name="VALUE" x="15.875" y="45.085" size="1.778" layer="96"/>
+</instance>
+<instance part="SUPPLY2" gate="GND" x="12.7" y="73.66" smashed="yes">
+<attribute name="VALUE" x="10.795" y="70.485" size="1.778" layer="96"/>
+</instance>
+<instance part="SUPPLY3" gate="GND" x="101.6" y="20.32" smashed="yes">
+<attribute name="VALUE" x="99.695" y="17.145" size="1.778" layer="96"/>
 </instance>
 </instances>
@@
 <label x="116.84" y="43.18" size="1.778" layer="95"/>
 </segment>
+<segment>
+<wire x1="144.78" y1="68.58" x2="137.16" y2="68.58" width="0.1524" layer="91"/>
+<pinref part="J4" gate="G$1" pin="9"/>
+<label x="139.7" y="68.58" size="1.778" layer="95"/>
+</segment>
 </net>
 <net name="5V" class="0">
+<segment>
+<pinref part="U1" gate="U1" pin="VCC"/>
+<wire x1="33.02" y1="81.28" x2="22.86" y2="81.28" width="0.1524" layer="91"/>
+<label x="22.86" y="81.28" size="1.778" layer="95"/>
+</segment>
+<segment>
+<wire x1="144.78" y1="43.18" x2="137.16" y2="43.18" width="0.1524" layer="91"/>
+<pinref part="J2" gate="J1" pin="2"/>
+<label x="139.7" y="43.18" size="1.778" layer="95"/>
+</segment>
+<segment>
+<wire x1="144.78" y1="60.96" x2="137.16" y2="60.96" width="0.1524" layer="91"/>
+<pinref part="J4" gate="G$1" pin="12"/>
+<label x="139.7" y="60.96" size="1.778" layer="95"/>
+</segment>
+<segment>
+<wire x1="144.78" y1="71.12" x2="137.16" y2="71.12" width="0.1524" layer="91"/>
+<pinref part="J4" gate="G$1" pin="8"/>
+<label x="139.7" y="71.12" size="1.778" layer="95"/>
+</segment>
 <segment>
 <pinref part="U1" gate="U1" pin="AVCC"/>
@@
 </segment>
 <segment>
-<pinref part="U1" gate="U1" pin="VCC"/>
-<wire x1="33.02" y1="81.28" x2="22.86" y2="81.28" width="0.1524" layer="91"/>
-<label x="22.86" y="81.28" size="1.778" layer="95"/>
-</segment>
-<segment>
-<wire x1="144.78" y1="43.18" x2="137.16" y2="43.18" width="0.1524" layer="91"/>
-<pinref part="J2" gate="J1" pin="2"/>
-<label x="139.7" y="43.18" size="1.778" layer="95"/>
+<pinref part="C1" gate="G$1" pin="+"/>
+<wire x1="12.7" y1="83.82" x2="12.7" y2="86.36" width="0.1524" layer="91"/>
+<label x="12.7" y="86.36" size="1.778" layer="95"/>
 </segment>
 </net>
@@
 <label x="22.86" y="73.66" size="1.778" layer="95"/>
 </segment>
+<segment>
+<wire x1="144.78" y1="66.04" x2="137.16" y2="66.04" width="0.1524" layer="91"/>
+<pinref part="J4" gate="G$1" pin="10"/>
+<label x="139.7" y="66.04" size="1.778" layer="95"/>
+</segment>
 </net>
 <net name="XTAL1" class="0">
 <segment>
 <pinref part="U1" gate="U1" pin="PB6(XTAL1/TOSC1)"/>
-<wire x1="33.02" y1="63.5" x2="22.86" y2="63.5" width="0.1524" layer="91"/>
+<wire x1="33.02" y1="63.5" x2="15.24" y2="63.5" width="0.1524" layer="91"/>
 <label x="22.86" y="63.5" size="1.778" layer="95"/>
+<pinref part="Y1" gate="G$1" pin="1"/>
+<wire x1="15.24" y1="58.42" x2="15.24" y2="63.5" width="0.1524" layer="91"/>
 </segment>
 </net>
@@
 <segment>
 <pinref part="U1" gate="U1" pin="PB7(XTAL2/TOSC2)"/>
-<wire x1="33.02" y1="58.42" x2="22.86" y2="58.42" width="0.1524" layer="91"/>
+<wire x1="33.02" y1="58.42" x2="20.32" y2="58.42" width="0.1524" layer="91"/>
 <label x="22.86" y="58.42" size="1.778" layer="95"/>
+<pinref part="Y1" gate="G$1" pin="3"/>
 </segment>
 </net>
@@
 <label x="139.7" y="45.72" size="1.778" layer="95"/>
 </segment>
+<segment>
+<wire x1="144.78" y1="73.66" x2="137.16" y2="73.66" width="0.1524" layer="91"/>
+<pinref part="J4" gate="G$1" pin="7"/>
+<label x="139.7" y="73.66" size="1.778" layer="95"/>
+</segment>
+<segment>
+<wire x1="144.78" y1="63.5" x2="137.16" y2="63.5" width="0.1524" layer="91"/>
+<pinref part="J4" gate="G$1" pin="11"/>
+<label x="139.7" y="63.5" size="1.778" layer="95"/>
+</segment>
+<segment>
+<pinref part="Y1" gate="G$1" pin="2"/>
+<pinref part="SUPPLY1" gate="GND" pin="GND"/>
+</segment>
+<segment>
+<pinref part="C1" gate="G$1" pin="-"/>
+<pinref part="SUPPLY2" gate="GND" pin="GND"/>
+</segment>
+<segment>
+<pinref part="D1" gate="D1" pin="C"/>
+<pinref part="SUPPLY3" gate="GND" pin="GND"/>
+</segment>
 </net>
 <net name="A0" class="0">
@@
 <label x="139.7" y="86.36" size="1.778" layer="95"/>
 </segment>
+<segment>
+<wire x1="144.78" y1="58.42" x2="137.16" y2="58.42" width="0.1524" layer="91"/>
+<pinref part="J4" gate="G$1" pin="13"/>
+<label x="139.7" y="58.42" size="1.778" layer="95"/>
+</segment>
 </net>
 <net name="A5" class="0">
@@
 <label x="139.7" y="88.9" size="1.778" layer="95"/>
 </segment>
+<segment>
+<wire x1="144.78" y1="55.88" x2="137.16" y2="55.88" width="0.1524" layer="91"/>
+<pinref part="J4" gate="G$1" pin="14"/>
+<label x="139.7" y="55.88" size="1.778" layer="95"/>
+</segment>
 </net>
 <net name="D0" class="0">
@@
 <wire x1="76.2" y1="30.48" x2="86.36" y2="30.48" width="0.1524" layer="91"/>
 <label x="78.74" y="30.48" size="1.778" layer="95"/>
+<pinref part="R1" gate="G$1" pin="1"/>
 </segment>
 <segment>
@@
 </segment>
 </net>
-<net name="N$21" class="0">
-<segment>
-<wire x1="144.78" y1="73.66" x2="137.16" y2="73.66" width="0.1524" layer="91"/>
-<pinref part="J4" gate="G$1" pin="7"/>
-</segment>
-</net>
-<net name="N$22" class="0">
-<segment>
-<wire x1="144.78" y1="71.12" x2="137.16" y2="71.12" width="0.1524" layer="91"/>
-<pinref part="J4" gate="G$1" pin="8"/>
-</segment>
-</net>
-<net name="N$23" class="0">
-<segment>
-<wire x1="144.78" y1="68.58" x2="137.16" y2="68.58" width="0.1524" layer="91"/>
-<pinref part="J4" gate="G$1" pin="9"/>
-</segment>
-</net>
-<net name="N$24" class="0">
-<segment>
-<wire x1="144.78" y1="66.04" x2="137.16" y2="66.04" width="0.1524" layer="91"/>
-<pinref part="J4" gate="G$1" pin="10"/>
-</segment>
-</net>
-<net name="N$25" class="0">
-<segment>
-<wire x1="144.78" y1="63.5" x2="137.16" y2="63.5" width="0.1524" layer="91"/>
-<pinref part="J4" gate="G$1" pin="11"/>
-</segment>
-</net>
-<net name="N$26" class="0">
-<segment>
-<wire x1="144.78" y1="60.96" x2="137.16" y2="60.96" width="0.1524" layer="91"/>
-<pinref part="J4" gate="G$1" pin="12"/>
-</segment>
-</net>
-<net name="N$27" class="0">
-<segment>
-<wire x1="144.78" y1="58.42" x2="137.16" y2="58.42" width="0.1524" layer="91"/>
-<pinref part="J4" gate="G$1" pin="13"/>
-</segment>
-</net>
-<net name="N$28" class="0">
-<segment>
-<wire x1="144.78" y1="55.88" x2="137.16" y2="55.88" width="0.1524" layer="91"/>
-<pinref part="J4" gate="G$1" pin="14"/>
-</segment>
-</net>
 <net name="N$5" class="0">
 <segment>
@@
 </segment>
 </net>
+<net name="N$2" class="0">
+<segment>
+<pinref part="R1" gate="G$1" pin="2"/>
+<pinref part="D1" gate="D1" pin="A"/>
+<wire x1="101.6" y1="30.48" x2="96.52" y2="30.48" width="0.1524" layer="91"/>
+</segment>
+</net>
